File: daughterboard/inputs.kicad_sch (KiCad schematic)
At the start: 66 parts, among them U8 LMV321IDBVR, U9 MAX9926UAEE+

Commit message: Rev 0.5 daughterboard, rev 0.6 1989-93/1994-95 motherboards: review fixes
Daughterboard rev 0.5:
- SN74LVC4245A drives the eight AUIPS2041 low sides at 5 V; output enable pulled
  off (R71) until the firmware enables it on PA8.
- BOOT1 pull-down (R72); hall input clamps D13/D14.
- ULN2003 COM to an SMAJ33A TVS (D11) instead of +12V: no key-off back-feed,
  no conduction in a 35 V load dump.
- Logic supply: D7/D8 -> 0.5 A PTC F1 -> SMAJ33A D12; C16 50 V, SS36 D9, C59.
- Tach stays an output.

Motherboards:
- Idle/VVT freewheel diodes, 4.7k switch pull-up options (not fitted),
  AUX VBAT PTC on all years.
- 1989-93 rev 0.6: two drivers per injector wire (0R links), SMCJ40A clamps.
- 2001-05: J1 3B tied to 3A.

Firmware: low-side enable (inverted open drain, forced writes, off during
configuration changes), unused control pins parked with pull-down, 1989-93
batch on all four outputs, VBATT offset noted.

Verification: 18/18 board tests, 119/119 harness check, circuit sims
20 OK / 3 CHECK / 6 REF / 0 FAIL, flash sim 9/9, firmware and bootloader
build; all boards 0 unconnected, 0 clearance errors.

Co-Authored-By: Claude Opus 5.5 <noreply@anthropic.com>
Claude-Session: https://claude.ai/code/session_012UFcA8PhPqkqYxcgEjD2n9
Parts:
- added D13, D14: 1N4148WS, Diode_SMD:D_SOD-323, symbol Device:D
Connections:
- net +3V3: now also D13.1 (K), D14.1 (K)
- net HALL1: now also D13.2 (A)
- net HALL2: now also D14.2 (A)

Commit message: Daughterboard rev 0.5b: in-stock parts for JLCPCB assembly
JLCPCB's BOM check flagged ten lines short of stock and one footprint mismatch.
All replacements are in stock at JLCPCB and fit the existing footprints (no re-route):
- Q1-Q8: onsemi NCV8406ASTT3G (C459816) instead of AUIPS2041LTR: same SOT-223
  pinout, 60-70 V active clamp, current limit, thermal shutdown, AEC-Q101.
- D11/D12 Littelfuse SMAJ33A (C223988); F1 TECHFUSE nSMD050-33V (C70077);
  L1 FH CMI322513U2R2KT (C70960); LEDs KENTO KT-0603G/B/Y; C103 YAGEO 33 nF
  50 V (C106862); R110 62 ohm 1% (C23222, was 61.9).
- U9 (MAX9926, spare VR inputs, out of stock everywhere) not fitted.
- U105 footprint renamed SOT-23-5 (AD8628ARTZ; pads identical to TSOT-23-5).
- JLC BOM: one line per LCSC part (SW1/SW2); not-fitted parts excluded.

Re-checked: netlist 754 pads 0 differences, DRC 0 unconnected / 0 clearance,
circuit sims with the NCV8406A model 20 OK / 3 CHECK / 6 REF / 0 FAIL.

Co-Authored-By: Claude Opus 5.5 <noreply@anthropic.com>
Claude-Session: https://claude.ai/code/session_012UFcA8PhPqkqYxcgEjD2n9
Parts:
- U9: Note dual VR conditioner (crank/cam) -> dual VR conditioner (spare VR inputs; not fitted)

Commit message: Daughterboard rev 0.5b: LM2903 VR conditioner, JLC placement fix, parts-availability swaps
- U9: the out-of-stock, single-source MAX9926 is replaced by an LM2903 dual comparator (TI, onsemi, UMW, ST...).
  Each VR input gets a BAT54S clamp to GND/+5V and 100k to a 1.65 V bias, each output 1M of hysteresis
  (D15-D18, R73-R80, C60). Same output polarity, so J2 wiring and firmware are unchanged. circuit_sim.py
  section H covers it (25 OK / 4 CHECK / 6 REF / 0 FAIL).
- Re-routed; daughter_patch_05b.py (with hand_route.py) routes HALL1, which the autorouter left open, and
  moves AN_AUX3 clear of the new clamps. Netlist 778 pads, 0 differences; DRC 0 unconnected, 0 clearance.
- CPLs for all boards now use the gerbers' own coordinates, with JLC's per-package rotation offsets
  (SOT-223/TO-252/SOT-23 +180, SOIC/TSSOP/LQFP +270, resistor arrays +90).
- Parts-availability review swaps: motherboard F4 to TECHFUSE nSMD050-33V (C70077; the old PTC is out of
  stock), D6 to Littelfuse SMCJ30A, D9 to Diodes B360A. MPX5700AP (NRND), the harness headers and the
  STM32F042 are recorded as supply open items in VERIFICATION.md.
- Viewer assets and README renders rebuilt.

Co-Authored-By: Claude Opus 5.5 <noreply@anthropic.com>
Claude-Session: https://claude.ai/code/session_012UFcA8PhPqkqYxcgEjD2n9
Parts:
- removed U9: MAX9926UAEE+, Package_SO:QSOP-16_3.9x4.9mm_P0.635mm, symbol ECU:MAX9926UAEE+
- added C60: 100n, Capacitor_SMD:C_0402_1005Metric, symbol Device:C
- added D15, D16, D17, D18: BAT54S, Package_TO_SOT_SMD:SOT-23, symbol Diode:BAT54S
- added R73, R74, R75, R76: 100k, Resistor_SMD:R_0402_1005Metric, symbol Device:R
- added R77, R78: 1M, Resistor_SMD:R_0402_1005Metric, symbol Device:R
- added R79, R80: 10k, Resistor_SMD:R_0402_1005Metric, symbol Device:R
- added U9: LM2903DR, Package_SO:SOIC-8_3.9x4.9mm_P1.27mm, symbol ECU:LM2903DR
Connections:
- net +3V3: now also R79.1
- net +5V: now also D15.2 (K), D16.2 (K), D17.2 (K), D18.2 (K), U9.8 (V+)
- net GND: now also C60.2, D15.1 (A), D16.1 (A), D17.1 (A), D18.1 (A), R80.2, U9.4 (GND)
- net VR1_INN: now also D16.3 (COM), R74.1, U9.6 (IN B-)
- net VR1_INP: now also D15.3 (COM), R73.1, R77.2, U9.5 (IN B+)
- net VR1_OUT: now also R77.1, U9.7 (OUT B)
- net VR2_INN: now also D18.3 (COM), R76.1, U9.2 (IN A-)
- net VR2_INP: now also D17.3 (COM), R75.1, R78.2, U9.3 (IN A+)
- net VR2_OUT: now also R78.1, U9.1 (OUT A)
- new net VR_BIAS: C60.1, R73.2, R74.2, R75.2, R76.2, R79.2, R80.1
- no-connect marks 2 -> 0
Other:
- note added: "Crank / cam VR inputs (spare): LM2903 comparator, 1M hysteresis, BAT54S clamps, biased to 1.65 V"
- note added: "VR input clamps, bias and hysteresis"
- note removed: "Crank / cam VR inputs: MAX9926 (outputs inverted, so harness + goes to IN-)"
