File: daughterboard/miata_ecu_daughter.kicad_sch (KiCad schematic)
At the start: 0 parts

Commit message: IAT source jumper on every motherboard; wideband MCU flashed through the main MCU
- motherboards (1989-93 / 1994-95 rev 0.5, 1996-97 / 1999-2000 / 2001-05
  rev 0.3): the R4/R5 0R links are replaced by JP1, a 1x3 2.54 mm header with
  a removable shunt (STOCK = harness sensor, EXT = IAT connector, default)
- daughterboard rev 0.4: USART3 (PD8/PD9) to the STM32F042's ROM-bootloader
  USART1 (PA9/PA10), plus PD10 -> its BOOT0 and PD11 -> its NRST, so both
  MCUs can be flashed over the one USB-C port (rusEFI support to be written;
  SWD pads kept as a fallback)
- scripts: schematic check now also catches nets split across sheets;
  motherboard project template bundled
- README: flashing and IAT sections

Co-Authored-By: Claude Opus 5.5 <noreply@anthropic.com>
Claude-Session: https://claude.ai/code/session_012UFcA8PhPqkqYxcgEjD2n9
Other:
- note added: "Miata ECU daughterboard rev 0.4 (on-board wideband controller, flashed through the main MCU). Block sheets connect through global labels; GND, +3V3, +5V and +12V are power symbols. J1 = power in and outputs (top edge), J2 = inputs and comms (bottom edge). 4-layer board: In1 GND plane, In2 +3V3 plane."
- note removed: "Miata ECU daughterboard rev 0.3 (on-board wideband controller). Block sheets connect through global labels; GND, +3V3, +5V and +12V are power symbols. J1 = power in and outputs (top edge), J2 = inputs and comms (bottom edge). 4-layer board: In1 GND plane, In2 +3V3 plane."

Commit message: Rev 0.5 daughterboard, rev 0.6 1989-93/1994-95 motherboards: review fixes
Daughterboard rev 0.5:
- SN74LVC4245A drives the eight AUIPS2041 low sides at 5 V; output enable pulled
  off (R71) until the firmware enables it on PA8.
- BOOT1 pull-down (R72); hall input clamps D13/D14.
- ULN2003 COM to an SMAJ33A TVS (D11) instead of +12V: no key-off back-feed,
  no conduction in a 35 V load dump.
- Logic supply: D7/D8 -> 0.5 A PTC F1 -> SMAJ33A D12; C16 50 V, SS36 D9, C59.
- Tach stays an output.

Motherboards:
- Idle/VVT freewheel diodes, 4.7k switch pull-up options (not fitted),
  AUX VBAT PTC on all years.
- 1989-93 rev 0.6: two drivers per injector wire (0R links), SMCJ40A clamps.
- 2001-05: J1 3B tied to 3A.

Firmware: low-side enable (inverted open drain, forced writes, off during
configuration changes), unused control pins parked with pull-down, 1989-93
batch on all four outputs, VBATT offset noted.

Verification: 18/18 board tests, 119/119 harness check, circuit sims
20 OK / 3 CHECK / 6 REF / 0 FAIL, flash sim 9/9, firmware and bootloader
build; all boards 0 unconnected, 0 clearance errors.

Co-Authored-By: Claude Opus 5.5 <noreply@anthropic.com>
Claude-Session: https://claude.ai/code/session_012UFcA8PhPqkqYxcgEjD2n9
Other:
- note added: "Miata ECU daughterboard rev 0.5 (on-board wideband controller, flashed through the main MCU; 5 V low-side drive, fused logic supply). Block sheets connect through global labels; GND, +3V3, +5V and +12V are power symbols. J1 = power in and outputs (top edge), J2 = inputs and comms (bottom edge). 4-layer board: In1 GND plane, In2 +3V3 plane."
- note removed: "Miata ECU daughterboard rev 0.4 (on-board wideband controller, flashed through the main MCU). Block sheets connect through global labels; GND, +3V3, +5V and +12V are power symbols. J1 = power in and outputs (top edge), J2 = inputs and comms (bottom edge). 4-layer board: In1 GND plane, In2 +3V3 plane."
