File: daughterboard/outputs.kicad_sch (KiCad schematic)
At the start: 26 parts, among them Q1 AUIPS2041LTR, Q2 AUIPS2041LTR, Q3 AUIPS2041LTR, Q4 AUIPS2041LTR, Q5 AUIPS2041LTR, Q6 AUIPS2041LTR, Q7 AUIPS2041LTR, Q8 AUIPS2041LTR, U5 ULN2003AD, U6 TC4427, U7 TC4427

Commit message: Rev 0.5 daughterboard, rev 0.6 1989-93/1994-95 motherboards: review fixes
Daughterboard rev 0.5:
- SN74LVC4245A drives the eight AUIPS2041 low sides at 5 V; output enable pulled
  off (R71) until the firmware enables it on PA8.
- BOOT1 pull-down (R72); hall input clamps D13/D14.
- ULN2003 COM to an SMAJ33A TVS (D11) instead of +12V: no key-off back-feed,
  no conduction in a 35 V load dump.
- Logic supply: D7/D8 -> 0.5 A PTC F1 -> SMAJ33A D12; C16 50 V, SS36 D9, C59.
- Tach stays an output.

Motherboards:
- Idle/VVT freewheel diodes, 4.7k switch pull-up options (not fitted),
  AUX VBAT PTC on all years.
- 1989-93 rev 0.6: two drivers per injector wire (0R links), SMCJ40A clamps.
- 2001-05: J1 3B tied to 3A.

Firmware: low-side enable (inverted open drain, forced writes, off during
configuration changes), unused control pins parked with pull-down, 1989-93
batch on all four outputs, VBATT offset noted.

Verification: 18/18 board tests, 119/119 harness check, circuit sims
20 OK / 3 CHECK / 6 REF / 0 FAIL, flash sim 9/9, firmware and bootloader
build; all boards 0 unconnected, 0 clearance errors.

Co-Authored-By: Claude Opus 5.5 <noreply@anthropic.com>
Claude-Session: https://claude.ai/code/session_012UFcA8PhPqkqYxcgEjD2n9
Parts:
- added C57, C58: 100n, Capacitor_SMD:C_0402_1005Metric, symbol Device:C
- added D11: SMAJ33A, Diode_SMD:D_SMA, symbol Device:D_Zener
- added R71: 10k, Resistor_SMD:R_0402_1005Metric, symbol Device:R
- added U11: SN74LVC4245APWR, Package_SO:TSSOP-24_4.4x7.8mm_P0.65mm, symbol ECU:SN74LVC4245APWR
- Q1, Q2, Q3, Q4, Q5, Q6, Q7, Q8: Note protected low side, 39V clamp -> protected low side, 63-75 V clamp
Connections:
- net +5V: now also C57.1, R71.1, U11.1 (VCCA)
- net ALT_CTL: now also U11.21 (B1); no longer Q8.1 (IN), R26.1
- net BOOST_CTL: now also U11.20 (B2); no longer Q7.1 (IN), R25.1
- net GND: now also C57.2, C58.2, D11.2 (A), U11.11 (GND), U11.12 (GND), U11.13 (GND), U11.2 (DIR)
- net IACV_CTL: now also U11.18 (B4); no longer Q5.1 (IN), R23.1
- net INJ1_CTL: now also U11.14 (B8); no longer Q1.1 (IN), R19.1
- net INJ2_CTL: now also U11.15 (B7); no longer Q2.1 (IN), R20.1
- net INJ3_CTL: now also U11.16 (B6); no longer Q3.1 (IN), R21.1
- net INJ4_CTL: now also U11.17 (B5); no longer Q4.1 (IN), R22.1
- net VVT_CTL: now also U11.19 (B3); no longer Q6.1 (IN), R24.1
- net +12V renamed ULN_COM
- net ULN_COM: now also D11.1 (K)
- new net +3V3: C58.1, U11.23 (VCCB), U11.24 (VCCB)
- new net ALT_IN: Q8.1 (IN), R26.1, U11.3 (A1)
- new net BOOST_IN: Q7.1 (IN), R25.1, U11.4 (A2)
- new net DRV_EN_N: R71.2, U11.22 (~{OE})
- new net IACV_IN: Q5.1 (IN), R23.1, U11.6 (A4)
- new net INJ1_IN: Q1.1 (IN), R19.1, U11.10 (A8)
- new net INJ2_IN: Q2.1 (IN), R20.1, U11.9 (A7)
- new net INJ3_IN: Q3.1 (IN), R21.1, U11.8 (A6)
- new net INJ4_IN: Q4.1 (IN), R22.1, U11.7 (A5)
- new net VVT_IN: Q6.1 (IN), R24.1, U11.5 (A3)
Other:
- note added: "3.3 V -> 5 V level shifter for the low-side inputs (DIR low: B -> A)"
- note added: "COM is not tied to +12V: a battery-fed relay coil cannot back-feed the ECU with the key off"
- note added: "Relay, lamp and tach outputs (ULN2003; flyback clamp: SMAJ33A TVS on COM)"
- note added: "~OE pulled up: all eight drivers off until the firmware drives DRV_EN_N low"
- note removed: "Relay, lamp and tach outputs (ULN2003, flyback to +12V)"

Commit message: Daughterboard rev 0.5b: in-stock parts for JLCPCB assembly
JLCPCB's BOM check flagged ten lines short of stock and one footprint mismatch.
All replacements are in stock at JLCPCB and fit the existing footprints (no re-route):
- Q1-Q8: onsemi NCV8406ASTT3G (C459816) instead of AUIPS2041LTR: same SOT-223
  pinout, 60-70 V active clamp, current limit, thermal shutdown, AEC-Q101.
- D11/D12 Littelfuse SMAJ33A (C223988); F1 TECHFUSE nSMD050-33V (C70077);
  L1 FH CMI322513U2R2KT (C70960); LEDs KENTO KT-0603G/B/Y; C103 YAGEO 33 nF
  50 V (C106862); R110 62 ohm 1% (C23222, was 61.9).
- U9 (MAX9926, spare VR inputs, out of stock everywhere) not fitted.
- U105 footprint renamed SOT-23-5 (AD8628ARTZ; pads identical to TSOT-23-5).
- JLC BOM: one line per LCSC part (SW1/SW2); not-fitted parts excluded.

Re-checked: netlist 754 pads 0 differences, DRC 0 unconnected / 0 clearance,
circuit sims with the NCV8406A model 20 OK / 3 CHECK / 6 REF / 0 FAIL.

Co-Authored-By: Claude Opus 5.5 <noreply@anthropic.com>
Claude-Session: https://claude.ai/code/session_012UFcA8PhPqkqYxcgEjD2n9
Parts:
- removed Q1, Q2, Q3, Q4, Q5, Q6, Q7, Q8: AUIPS2041LTR, Package_TO_SOT_SMD:SOT-223, symbol ECU:AUIPS2041LTR
- added Q1, Q2, Q3, Q4, Q5, Q6, Q7, Q8: NCV8406ASTT3G, Package_TO_SOT_SMD:SOT-223, symbol ECU:NCV8406ASTT3G
- D11: LCSC C3720609 -> C223988; Note TVS: ULN2003 flyback clamp (Bourns) -> TVS: ULN2003 flyback clamp (Littelfuse)
Connections:
- net ALT_IN: now also Q8.1 (G)
- net BOOST_IN: now also Q7.1 (G)
- net GND: now also Q1.3 (S), Q2.3 (S), Q3.3 (S), Q4.3 (S), Q5.3 (S), Q6.3 (S), Q7.3 (S), Q8.3 (S)
- net IACV_IN: now also Q5.1 (G)
- net INJ1_IN: now also Q1.1 (G)
- net INJ2_IN: now also Q2.1 (G)
- net INJ3_IN: now also Q3.1 (G)
- net INJ4_IN: now also Q4.1 (G)
- net OUT_ALT: now also Q8.2 (D), Q8.4 (D)
- net OUT_BOOST: now also Q7.2 (D), Q7.4 (D)
- net OUT_IACV: now also Q5.2 (D), Q5.4 (D)
- net OUT_INJ1: now also Q1.2 (D), Q1.4 (D)
- net OUT_INJ2: now also Q2.2 (D), Q2.4 (D)
- net OUT_INJ3: now also Q3.2 (D), Q3.4 (D)
- net OUT_INJ4: now also Q4.2 (D), Q4.4 (D)
- net OUT_VVT: now also Q6.2 (D), Q6.4 (D)
- net VVT_IN: now also Q6.1 (G)
Other:
- note added: "Protected low-side drivers (NCV8406A): injectors, IACV, VVT, boost, alternator"
- note removed: "Protected low-side drivers (AUIPS2041L): injectors, IACV, VVT, boost, alternator"
