File: daughterboard/power.kicad_sch (KiCad schematic)
At the start: 32 parts, among them U2 LMR14020, U3 TLS115B0EJ, U4 AMS1117-3.3

Commit message: Rev 0.5 daughterboard, rev 0.6 1989-93/1994-95 motherboards: review fixes
Daughterboard rev 0.5:
- SN74LVC4245A drives the eight AUIPS2041 low sides at 5 V; output enable pulled
  off (R71) until the firmware enables it on PA8.
- BOOT1 pull-down (R72); hall input clamps D13/D14.
- ULN2003 COM to an SMAJ33A TVS (D11) instead of +12V: no key-off back-feed,
  no conduction in a 35 V load dump.
- Logic supply: D7/D8 -> 0.5 A PTC F1 -> SMAJ33A D12; C16 50 V, SS36 D9, C59.
- Tach stays an output.

Motherboards:
- Idle/VVT freewheel diodes, 4.7k switch pull-up options (not fitted),
  AUX VBAT PTC on all years.
- 1989-93 rev 0.6: two drivers per injector wire (0R links), SMCJ40A clamps.
- 2001-05: J1 3B tied to 3A.

Firmware: low-side enable (inverted open drain, forced writes, off during
configuration changes), unused control pins parked with pull-down, 1989-93
batch on all four outputs, VBATT offset noted.

Verification: 18/18 board tests, 119/119 harness check, circuit sims
20 OK / 3 CHECK / 6 REF / 0 FAIL, flash sim 9/9, firmware and bootloader
build; all boards 0 unconnected, 0 clearance errors.

Co-Authored-By: Claude Opus 5.5 <noreply@anthropic.com>
Claude-Session: https://claude.ai/code/session_012UFcA8PhPqkqYxcgEjD2n9
Parts:
- added C59: 10u, Capacitor_SMD:C_0805_2012Metric, symbol Device:C
- added D12: SMAJ33A, Diode_SMD:D_SMA, symbol Device:D_Zener
- added F1: SMD1206P050TF/24, Fuse:Fuse_1206_3216Metric, symbol Device:Fuse
- C16: value 4.7u -> 10u/50V; footprint Capacitor_SMD:C_0603_1608Metric -> Capacitor_SMD:C_1206_3216Metric; LCSC C19666 -> C13585
- D9: value SS34 -> SS36; LCSC C8678 -> C7428237; Note catch diode -> catch diode, 60 V 3 A SMA (rev 0.5)
Connections:
- net +12V: now also D12.1 (K), F1.2; no longer D7.1 (K), D8.1 (K)
- net +5V: now also C59.1
- net GND: now also C59.2, D12.2 (A)
- new net +12V_IN: D7.1 (K), D8.1 (K), F1.1
Other:
- note added: "Input protection (fused, TVS-clamped logic supply) and 5 V buck (LMR14020, 5 V / 2 A)"
- note removed: "Input protection and 5 V buck (LMR14020, 5 V / 2 A)"

Commit message: Daughterboard: 5.5 A buck inductor, 33 pF crystal caps; NB alternator control off by default
- L2: Sunlord MWSA0603S-100MT (C132141, 10 uH, Isat 5.5 A, 7 x 6.6 mm). The
  MWSA0503S saturated at 3.5 A, below the LMR14020's 3.8 A maximum current
  limit. Placed on end; D9 and the feedback divider moved 0.3 mm left.
- C13/C14: 33 pF C0G (C1663) for the 20 pF crystal (were 22 pF).
- Firmware: NB alternator control ships off until the field current is
  measured (pin, PID and target still set up). Test checks the field isn't
  driven with the default tune.
- Daughterboard re-routed and released: 754 pads match, 0 unconnected,
  0 clearance errors. Viewer assets and README renders refreshed.

Co-Authored-By: Claude Opus 5.5 <noreply@anthropic.com>
Claude-Session: https://claude.ai/code/session_012UFcA8PhPqkqYxcgEjD2n9
Parts:
- L2: footprint Inductor_SMD:L_Sunlord_MWSA0503S -> Inductor_SMD:L_Sunlord_MWSA0603S; LCSC C139506 -> C132141; Note (none) -> buck inductor, Sunlord MWSA0603S-100MT

Commit message: Daughterboard rev 0.5b: in-stock parts for JLCPCB assembly
JLCPCB's BOM check flagged ten lines short of stock and one footprint mismatch.
All replacements are in stock at JLCPCB and fit the existing footprints (no re-route):
- Q1-Q8: onsemi NCV8406ASTT3G (C459816) instead of AUIPS2041LTR: same SOT-223
  pinout, 60-70 V active clamp, current limit, thermal shutdown, AEC-Q101.
- D11/D12 Littelfuse SMAJ33A (C223988); F1 TECHFUSE nSMD050-33V (C70077);
  L1 FH CMI322513U2R2KT (C70960); LEDs KENTO KT-0603G/B/Y; C103 YAGEO 33 nF
  50 V (C106862); R110 62 ohm 1% (C23222, was 61.9).
- U9 (MAX9926, spare VR inputs, out of stock everywhere) not fitted.
- U105 footprint renamed SOT-23-5 (AD8628ARTZ; pads identical to TSOT-23-5).
- JLC BOM: one line per LCSC part (SW1/SW2); not-fitted parts excluded.

Re-checked: netlist 754 pads 0 differences, DRC 0 unconnected / 0 clearance,
circuit sims with the NCV8406A model 20 OK / 3 CHECK / 6 REF / 0 FAIL.

Co-Authored-By: Claude Opus 5.5 <noreply@anthropic.com>
Claude-Session: https://claude.ai/code/session_012UFcA8PhPqkqYxcgEjD2n9
Parts:
- D12: LCSC C3720609 -> C223988; Note TVS on the fused logic supply (Bourns) -> TVS on the fused logic supply (Littelfuse)
- F1: value SMD1206P050TF/24 -> nSMD050-33V; LCSC C209741 -> C70077; Note PTC 0.5 A hold / 1 A trip, 24 V: logic supply fuse -> PTC 0.5 A hold / 1 A trip, 33 V: logic supply fuse
- L1: LCSC C223413 -> C70960; Note input filter (Taiyo Yuden LBC3225T2R2MR, 930 mA, 80 mOhm) -> input filter (FH CMI322513U2R2KT, 500 mA, 0.3 ohm)

Commit message: Daughterboard rev 0.5b: LM2903 VR conditioner, JLC placement fix, parts-availability swaps
- U9: the out-of-stock, single-source MAX9926 is replaced by an LM2903 dual comparator (TI, onsemi, UMW, ST...).
  Each VR input gets a BAT54S clamp to GND/+5V and 100k to a 1.65 V bias, each output 1M of hysteresis
  (D15-D18, R73-R80, C60). Same output polarity, so J2 wiring and firmware are unchanged. circuit_sim.py
  section H covers it (25 OK / 4 CHECK / 6 REF / 0 FAIL).
- Re-routed; daughter_patch_05b.py (with hand_route.py) routes HALL1, which the autorouter left open, and
  moves AN_AUX3 clear of the new clamps. Netlist 778 pads, 0 differences; DRC 0 unconnected, 0 clearance.
- CPLs for all boards now use the gerbers' own coordinates, with JLC's per-package rotation offsets
  (SOT-223/TO-252/SOT-23 +180, SOIC/TSSOP/LQFP +270, resistor arrays +90).
- Parts-availability review swaps: motherboard F4 to TECHFUSE nSMD050-33V (C70077; the old PTC is out of
  stock), D6 to Littelfuse SMCJ30A, D9 to Diodes B360A. MPX5700AP (NRND), the harness headers and the
  STM32F042 are recorded as supply open items in VERIFICATION.md.
- Viewer assets and README renders rebuilt.

Co-Authored-By: Claude Opus 5.5 <noreply@anthropic.com>
Claude-Session: https://claude.ai/code/session_012UFcA8PhPqkqYxcgEjD2n9
Parts:
- D6: LCSC C310046 -> C224048
- D9: value SS36 -> B360A; LCSC C7428237 -> C94193; Note catch diode, 60 V 3 A SMA (rev 0.5) -> catch diode, 60 V 3 A SMA (rev 0.5; Diodes B360A-13-F since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
