File: daughterboard/wideband.kicad_sch (KiCad schematic)
At the start: 57 parts, among them J102 SWD (WBO), Q101 VND14NV04, U101 MCP6004, U102 STM32F042K6T6, U103 REF3033, U105 AD8628, U106 SN65HVD230DR

Commit message: IAT source jumper on every motherboard; wideband MCU flashed through the main MCU
- motherboards (1989-93 / 1994-95 rev 0.5, 1996-97 / 1999-2000 / 2001-05
  rev 0.3): the R4/R5 0R links are replaced by JP1, a 1x3 2.54 mm header with
  a removable shunt (STOCK = harness sensor, EXT = IAT connector, default)
- daughterboard rev 0.4: USART3 (PD8/PD9) to the STM32F042's ROM-bootloader
  USART1 (PA9/PA10), plus PD10 -> its BOOT0 and PD11 -> its NRST, so both
  MCUs can be flashed over the one USB-C port (rusEFI support to be written;
  SWD pads kept as a fallback)
- scripts: schematic check now also catches nets split across sheets;
  motherboard project template bundled
- README: flashing and IAT sections

Co-Authored-By: Claude Opus 5.5 <noreply@anthropic.com>
Claude-Session: https://claude.ai/code/session_012UFcA8PhPqkqYxcgEjD2n9
Connections:
- net WB_PROG_RX: now reaches U102.19 (PA9)
- net WB_PROG_TX: now reaches U102.20 (PA10)
- no-connect marks 11 -> 9

Commit message: Daughterboard rev 0.5b: in-stock parts for JLCPCB assembly
JLCPCB's BOM check flagged ten lines short of stock and one footprint mismatch.
All replacements are in stock at JLCPCB and fit the existing footprints (no re-route):
- Q1-Q8: onsemi NCV8406ASTT3G (C459816) instead of AUIPS2041LTR: same SOT-223
  pinout, 60-70 V active clamp, current limit, thermal shutdown, AEC-Q101.
- D11/D12 Littelfuse SMAJ33A (C223988); F1 TECHFUSE nSMD050-33V (C70077);
  L1 FH CMI322513U2R2KT (C70960); LEDs KENTO KT-0603G/B/Y; C103 YAGEO 33 nF
  50 V (C106862); R110 62 ohm 1% (C23222, was 61.9).
- U9 (MAX9926, spare VR inputs, out of stock everywhere) not fitted.
- U105 footprint renamed SOT-23-5 (AD8628ARTZ; pads identical to TSOT-23-5).
- JLC BOM: one line per LCSC part (SW1/SW2); not-fitted parts excluded.

Re-checked: netlist 754 pads 0 differences, DRC 0 unconnected / 0 clearance,
circuit sims with the NCV8406A model 20 OK / 3 CHECK / 6 REF / 0 FAIL.

Co-Authored-By: Claude Opus 5.5 <noreply@anthropic.com>
Claude-Session: https://claude.ai/code/session_012UFcA8PhPqkqYxcgEjD2n9
Parts:
- C103: LCSC C285077 -> C106862
- R110: value 61.9 -> 62; LCSC C23092 -> C23222
- U105: footprint Package_TO_SOT_SMD:TSOT-23-5 -> Package_TO_SOT_SMD:SOT-23-5
