File: motherboards/1994-95/miata_mb_9495.kicad_pcb (KiCad board)
At the start: 2 copper layers, 154 x 161.5 mm, 29 parts, among them J1 TE 174917-6, J2 LSU 4.9, J3 IAT, J4 USB-C, J5 AUX 2x8, U2 MPX5700AP, U4 USBLC6-2SC6

Commit message: IAT source jumper on every motherboard; wideband MCU flashed through the main MCU
- motherboards (1989-93 / 1994-95 rev 0.5, 1996-97 / 1999-2000 / 2001-05
  rev 0.3): the R4/R5 0R links are replaced by JP1, a 1x3 2.54 mm header with
  a removable shunt (STOCK = harness sensor, EXT = IAT connector, default)
- daughterboard rev 0.4: USART3 (PD8/PD9) to the STM32F042's ROM-bootloader
  USART1 (PA9/PA10), plus PD10 -> its BOOT0 and PD11 -> its NRST, so both
  MCUs can be flashed over the one USB-C port (rusEFI support to be written;
  SWD pads kept as a fallback)
- scripts: schematic check now also catches nets split across sheets;
  motherboard project template bundled
- README: flashing and IAT sections

Co-Authored-By: Claude Opus 5.5 <noreply@anthropic.com>
Claude-Session: https://claude.ai/code/session_012UFcA8PhPqkqYxcgEjD2n9
Parts:
- removed R4, R5: 0R, Resistor_SMD:R_0603_1608Metric
- added JP1: IAT SEL, Connector_PinHeader_2.54mm:PinHeader_1x03_P2.54mm_Vertical, F.Cu at (152.5, 195.0)
Routing:
- net IN_IAT: track 60.6 -> 56.0 mm
- net IN_MAP: track 148.9 -> 151.2 mm, vias 1 -> 2
- net /LSU, MAP, IAT, USB, AUX/USB_CC1: track 8.16 -> 5.91 mm, vias 2 -> 0
- net HARN_IAT: track 175.9 -> 177.6 mm, vias 3 -> 4
- net LSU_UN: track 134.0 -> 132.4 mm, vias 2 -> 1
- net /LSU, MAP, IAT, USB, AUX/IAT_EXT: track 8.31 -> 6.91 mm, vias 1 -> 0
- net V5_SENS: track 305.7 -> 307.0 mm
- net OUT_IGN3: track 167.2 -> 168.1 mm
- net USB_VBUS: track 85.0 -> 85.6 mm
- net GND: vias 1084 -> 1067
Other:
- board text added: "EXT"
- board text added: "IAT"
- board text added: "Miata ECU motherboard 1994-1995 (NA8) rev 0.5"
- board text added: "STOCK"
- board text removed: "Miata ECU motherboard 1994-1995 (NA8) rev 0.4"

Commit message: Rev 0.5 daughterboard, rev 0.6 1989-93/1994-95 motherboards: review fixes
Daughterboard rev 0.5:
- SN74LVC4245A drives the eight AUIPS2041 low sides at 5 V; output enable pulled
  off (R71) until the firmware enables it on PA8.
- BOOT1 pull-down (R72); hall input clamps D13/D14.
- ULN2003 COM to an SMAJ33A TVS (D11) instead of +12V: no key-off back-feed,
  no conduction in a 35 V load dump.
- Logic supply: D7/D8 -> 0.5 A PTC F1 -> SMAJ33A D12; C16 50 V, SS36 D9, C59.
- Tach stays an output.

Motherboards:
- Idle/VVT freewheel diodes, 4.7k switch pull-up options (not fitted),
  AUX VBAT PTC on all years.
- 1989-93 rev 0.6: two drivers per injector wire (0R links), SMCJ40A clamps.
- 2001-05: J1 3B tied to 3A.

Firmware: low-side enable (inverted open drain, forced writes, off during
configuration changes), unused control pins parked with pull-down, 1989-93
batch on all four outputs, VBATT offset noted.

Verification: 18/18 board tests, 119/119 harness check, circuit sims
20 OK / 3 CHECK / 6 REF / 0 FAIL, flash sim 9/9, firmware and bootloader
build; all boards 0 unconnected, 0 clearance errors.

Co-Authored-By: Claude Opus 5.5 <noreply@anthropic.com>
Claude-Session: https://claude.ai/code/session_012UFcA8PhPqkqYxcgEjD2n9
Parts:
- added D1: SS34, Diode_SMD:D_SMA, F.Cu at (203.7, 102.0)
- added D2: SS34, Diode_SMD:D_SMA, F.Cu at (211.3, 102.0)
- added F4: 0.5A hold, Fuse:Fuse_1206_3216Metric, F.Cu at (198.0, 163.0)
- added R20: 4.7k, Resistor_SMD:R_0603_1608Metric, F.Cu at (163.1, 144.0)
- added R21: 4.7k, Resistor_SMD:R_0603_1608Metric, F.Cu at (165.6, 144.0)
- added R22: 4.7k, Resistor_SMD:R_0603_1608Metric, F.Cu at (168.1, 144.0)
Connections:
- J5 pad 15: VBAT_IN -> /LSU, MAP, IAT, USB, AUX/AUX_VBAT
Routing:
- net VBAT_IN: track 203.1 -> 351.4 mm, vias 6 -> 9
- net /LSU, MAP, IAT, USB, AUX/AUX_VBAT: track 0.00 -> 37.8 mm, vias 0 -> 3
- net OUT_VVT: track 33.1 -> 36.3 mm, vias 2 -> 3
- net OUT_IACV: track 33.7 -> 37.0 mm, vias 2 -> 3
- net IN_MAP: track 151.2 -> 148.7 mm, vias 2 -> 1
- net /LSU, MAP, IAT, USB, AUX/USB_CC1: track 5.91 -> 8.16 mm, vias 0 -> 2
- net USB_VBUS: track 85.6 -> 83.9 mm
- net V5_SENS: track 307.0 -> 305.5 mm
- net IN_SW3: track 91.5 -> 92.5 mm, vias 2 -> 3
- net IN_SW1: track 87.7 -> 88.4 mm, vias 2 -> 3
- net IN_SW2: track 84.2 -> 85.0 mm, vias 2 -> 3
- net OUT_MAINRLY: track 141.5 -> 142.1 mm, vias 2 -> 3
- net OUT_BOOST: track 118.9 -> 119.1 mm, vias 2 -> 3
- net GND: vias 1067 -> 1031
Other:
- board text added: "Miata ECU motherboard 1994-1995 (NA8) rev 0.6"
- board text removed: "Miata ECU motherboard 1994-1995 (NA8) rev 0.5"
